File: clackotron2000/clackotron2000.kicad_sch (KiCad schematic)
At the start: 58 parts, among them J3 Conn_ESP_Prog, J4 Power, J5 Output, J6 Conn_01x04, Q1 BSN20, Q2 BSN20, Q3 BSN20, Q4 BSN20, SW1 SW_Push_DPDT, SW2 SW_Push, SW3 SW_Push, U1 ESP32-WROOM-32, U2 SP3485EN, U3 R-78B5.0-1.0, U4 PCF85263ATT, U5 AMS1117-3.3, Y1 Crystal

Commit message: chore: rebase changes from internal repository
Parts:
- U3: digikey (none) -> R-78K5.0-0.5
Changed lines of the file:
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@@
+      (effects (font (size 1.27 1.27)) hide)
+    )
+    (property "digikey" "R-78K5.0-0.5" (at 182.88 31.75 0)
       (effects (font (size 1.27 1.27)) hide)
     )

Commit message: add new parts for next hardware revision to schematic
Parts:
- added C17, C18: 100nF, Capacitor_SMD:C_0805_2012Metric, symbol Device:C
- added C19: 1uF, Capacitor_SMD:C_0805_2012Metric, symbol Device:C
- added D7, D8, D9: LESD5D5.0CT1G, clackotron_fp:SOD-523_L1.2-W0.8-LS1.6-BI, symbol clackotronlib:LESD5D5.0CT1G
- added R19, R20, R21, R22, R23: 10k, Resistor_SMD:R_0805_2012Metric, symbol Device:R
- added SW4, SW5: K2-1102SP-C4SC-04, clackotron_fp:KEY-SMD_4P-L6.0-W6.0-P4.50-LS9.5-BL, symbol clackotronlib:K2-1102SP-C4SC-04
- added U6: ESP32-S3-WROOM-1(N8R2), clackotron_fp:WIRELM-SMD_ESP32-S3-WROOM-1, symbol clackotronlib:ESP32-S3-WROOM-1(N8R2)
- added USBC1: USB3.1C16PFSMT, clackotron_fp:USB-C-SMD_TYPE-C-USB-17, symbol clackotronlib:USB3.1C16PFSMT
Connections:
- net IO0 is gone; now on net Button1: J3.3 (Pin_3), U1.25 (IO0)
- net +3V3: now also C18.1, C19.1, R21.1, R22.1, R23.1, U6.2 (3V3)
- net Button1: now also R22.2, SW4.1, SW4.2, U6.27 (IO0)
- net Button2: now also R23.2, SW5.1, SW5.2, U6.26 (IO45)
- net DataEN: now also U6.10 (IO17)
- net DataRX: now also U6.9 (IO16)
- net DataTX: now also U6.11 (IO18)
- net EN: now also C17.1, R21.2, U6.3 (EN)
- net GND: now also C17.2, C18.2, C19.2, D7.1, D8.1, D9.1, R19.1, R20.2, SW4.3, SW4.4, SW5.3, SW5.4, U6.1 (GND), U6.40 (GND), U6.41 (GND), USBC1.0, USBC1.A1 (GND), USBC1.A12 (GND)
- net LED_Data: now also U6.8 (IO15)
- net RXD0: now also U6.36 (RXD0)
- net TXD0: now also U6.37 (TXD0)
- new net: D7.2, USBC1.A4 (VBUS), USBC1.A9 (VBUS)
- new net: R20.1, USBC1.A5 (CC1)
- new net: R19.2, USBC1.B5 (CC2)
- new net D+: D9.2, U6.14 (IO20), USBC1.A6 (DP1), USBC1.B6 (DP2)
- new net D-: D8.2, U6.13 (IO19), USBC1.A7 (DN1), USBC1.B7 (DN2)
- no-connect marks 19 -> 21

Commit message: hardware redesign for v3.0 done
Parts:
- removed C2, C3, C9: 100nF, Capacitor_SMD:C_0805_2012Metric, symbol Device:C
- removed C4: 1uF, Capacitor_SMD:C_0805_2012Metric, symbol Device:C
- removed D3, D5: LED, LED_SMD:LED_0805_2012Metric, symbol Device:LED
- removed D6: WS2812B, LED_SMD:LED_WS2812B_PLCC4_5.0x5.0mm_P3.2mm, symbol LED:WS2812B
- removed J6: Conn_01x04, Connector_JST:JST_SH_SM04B-SRSS-TB_1x04-1MP_P1.00mm_Horizontal, symbol Connector_Generic:Conn_01x04
- removed R1, R16, R2: 10k, Resistor_SMD:R_0805_2012Metric, symbol Device:R
- removed R5, R7: 1k1, Resistor_SMD:R_0805_2012Metric, symbol Device:R
- removed SW1: SW_Push_DPDT, clackotron_fp:SW_Push_DPDT, symbol Switch:SW_Push_DPDT
- removed SW2, SW3: SW_Push, JLCPCB:SW-SMD_4P-L6.0-W6.0-P4.50-LS10.0-BL, symbol Switch:SW_MEC_5E
- removed U1: ESP32-WROOM-32, RF_Module:ESP32-WROOM-32, symbol RF_Module:ESP32-WROOM-32
- added D7: 1N4007, Diode_SMD:D_SMA, symbol Diode:1N4001
- D2: renamed from D8; LCSC Part # (none) -> C383211
- D3: renamed from D9; LCSC Part # (none) -> C383211
- D5: renamed from D7; LCSC Part # (none) -> C383211
- J2: renamed from J4; LCSC Part # (none) -> C466970
- J3: renamed from J5; LCSC Part # (none) -> C98769
- R5: renamed from R19; value 10k -> 5.1k
- R6: renamed from R20; value 10k -> 5.1k
- SW1: renamed from SW4; LCSC Part # (none) -> C127509
- SW2: renamed from SW5; LCSC Part # (none) -> C127509
- U2: renamed from U6; LCSC Part # (none) -> C2913204
- U4: renamed from U3; digikey R-78K5.0-0.5 -> 945-R-78K5.0-1.0-ND
- USBC1: LCSC Part # (none) -> C167321
- renumbered C18 to C1, C12 to C11, C1 to C12, C7 to C2, C17 to C3, C6 to C4, C19 to C5, C5 to C6, C8 to C7, C16 to C8, C11 to C9, D2 to D4, D4 to D6, J3 to J1, R18 to R1, R23 to R10, R8 to R11, R9 to R12, R10 to R13, R11 to R14, R12 to R15, R13 to R16, R14 to R17, R15 to R18, R21 to R2, R22 to R7, R17 to R8, R6 to R9, U4 to U1, U2 to U3
Connections:
- net SCK is gone; now on net SCL: R3.2, U1.6 (SCL)
- net +5V: now also D7.1 (K)
- net +VDC: now also D4.1 (K)
- net DataRX: now also U2.11 (IO18); no longer U2.9 (IO16)
- net DataTX: now also U2.9 (IO16); no longer U2.11 (IO18)
- net SDA: now also U2.38 (IO2)
- net VBUS: now reaches D5.2, USBC1.A4 (VBUS), USBC1.A9 (VBUS)
- net VBUS: now also D7.2 (A)
- net SCL: now reaches U2.39 (IO1)
- no-connect marks 21 -> 27
Other:
- note removed: "Button1"
- note removed: "Button2"
- note removed: "Data Enable"
- note removed: "Data Rx"
- note removed: "Data Tx"
- note removed: "LED1"
- note removed: "LED2"
- note removed: "SCK"
- note removed: "SDA"
- moved on the sheet: BT1, C1, C12, C2, C3, C4, C5, C6, C7, D1, D2, D3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

Commit message: generate production data and fix some part numbers and stuff
Parts:
- J2, J3, U1: now in the parts list
Changed lines of the file:
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@@
   )
   (symbol (lib_id "Connector:Screw_Terminal_01x02") (at 133.985 34.29 180) (unit 1)
-    (in_bom no) (on_board yes) (dnp no)
+    (in_bom yes) (on_board yes) (dnp no)
     (property "Reference" "J2" (at 133.985 25.4 0)
       (effects (font (size 1.27 1.27)))
@@
   )
   (symbol (lib_id "Connector:Screw_Terminal_01x04") (at 142.24 50.8 0) (unit 1)
-    (in_bom no) (on_board yes) (dnp no) (fields_autoplaced)
+    (in_bom yes) (on_board yes) (dnp no) (fields_autoplaced)
     (property "Reference" "J3" (at 145.415 50.7999 0)
       (effects (font (size 1.27 1.27)) (justify left))
@@
   )
   (symbol (lib_id "Timer_RTC:PCF85263ATT") (at 52.07 149.225 0) (unit 1)
-    (in_bom no) (on_board yes) (dnp no)
+    (in_bom yes) (on_board yes) (dnp no)
     (property "Reference" "U1" (at 43.18 140.335 0)
       (effects (font (size 1.27 1.27)))

Commit message: add new parts. not yet done...
Parts:
- R11, R12, R13, R14: Manufacturer (none) -> C325794
- R9: LCSC Part (none) -> C17375; LCSC Part # C17375 -> C325794
- Y1: LCSC Part (none) -> C515342; LCSC Part # C515342 -> C130253
Changed lines of the file:
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@@
+      (effects (font (size 1.27 1.27)) hide)
+    )
+    (property "Manufacturer" "C325794" (at 227.965 95.885 0)
       (effects (font (size 1.27 1.27)) hide)
     )
@@
     )
     (property "LCSC Part #" "C17520" (at 227.965 68.58 0)
+      (effects (font (size 1.27 1.27)) hide)
+    )
+    (property "Manufacturer" "C325794" (at 227.965 68.58 0)
       (effects (font (size 1.27 1.27)) hide)
     )
@@
       (effects (font (size 1.27 1.27)) hide)
     )
-    (property "LCSC Part #" "C515342" (at 30.48 158.115 0)
+    (property "LCSC Part #" "C130253" (at 30.48 158.115 0)
+      (effects (font (size 1.27 1.27)) hide)
+    )
+    (property "LCSC Part" "C515342" (at 30.48 158.115 0)
       (effects (font (size 1.27 1.27)) hide)
     )
@@
       (effects (font (size 1.27 1.27)) hide)
     )
+    (property "Manufacturer" "C325794" (at 227.965 123.825 0)
+      (effects (font (size 1.27 1.27)) hide)
+    )
     (pin "1")
     (pin "2")
@@
       (effects (font (size 1.27 1.27)) hide)
     )
-    (property "LCSC Part #" "C17375" (at 193.04 35.56 0)
+    (property "LCSC Part #" "C325794" (at 193.04 35.56 0)
+      (effects (font (size 1.27 1.27)) hide)
+    )
+    (property "LCSC Part" "C17375" (at 193.04 35.56 0)
       (effects (font (size 1.27 1.27)) hide)
     )
@@
       (effects (font (size 1.27 1.27)) hide)
     )
+    (property "Manufacturer" "C325794" (at 227.965 151.13 0)
+      (effects (font (size 1.27 1.27)) hide)
+    )

Commit message: changed all parts. set to version 3.1
Parts:
- removed U1: PCF85263ATT, Package_SO:TSSOP-8_3x3mm_P0.65mm, symbol Timer_RTC:PCF85263ATT
- added U1: PCF85263ATL, Package_DFN_QFN:DFN-10-1EP_2.6x2.6mm_P0.5mm_EP1.3x2.2mm, symbol clackotronlib:PCF85263ATL
- J1, U4: now not fitted
Connections:
- net +3V3: now also U1.10 (VDD)
- net GND: now also U1.11 (GNDPAD), U1.5 (VSS)
- net SCL: now also U1.7 (SCL)
- net SDA: now also U1.6 (SDA)
- net at BT1.1 (+), C6.1: now also U1.3 (VBAT)
- net at R1.1: now also U1.1 (OSCI)
- net at Y1.2: now also U1.2 (OSCO)
- no-connect marks 27 -> 30
Other:
- moved on the sheet: BT1, C2, C4, C6, R1, Y1
